File: hardware/pc_max30003_brk.sch (EAGLE design)
At the start: 32 parts, among them U2 TXB0108PWR, U4 AP2112K-3.3V

Commit message: updated design file
Parts:
- removed JMP2: 0R-JUMPA, jump-0r-smd:0R-JUMPA
- U4: value AP2112K-3.3V -> AP2112K-1.8V
Connections:
- removed net +3V3: C12.2, C13.1, C14.1, C15.2, C4.1, C5.1, JMP2-0R.3, R1.1, SV1.3, U$1.AVDD, U$1.DVDD, U$1.OVDD, U2.VCCA, U4.OUT
- removed net VCC: C11.2, JMP2-0R.2, U2.VCCB
- new net +1.8V: C12.2, C13.1, C14.1, C15.2, C4.1, C5.1, R1.1, U$1.AVDD, U$1.DVDD, U$1.OVDD, U2.VCCA, U4.OUT
- net GND: now also SV1.3
- net VDD: now also C11.2, U2.VCCB; no longer JMP2-0R.1
Other:
- note added: "CONNECTOR"
- note added: "ECG"
- note added: "LOGIC LEVEL CONVERTER"
- note added: "POWER SUPPLY"
- moved on the sheet: C1, C10, C11, C12, C13, C14, C15, C16, C2, C3, C4, C5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
